Commit message: Added original spheres on atlas.

File: assets/atlas/atlas_convex_hull_hydro.urdf (robot description, URDF)
Before this commit: robot atlas, 68 links, 67 joints
Links:
- link l_foot: geometry collision mesh filename=./meshes/l_foot_chull.obj; visual mesh filename=./meshes/l_foot.obj
- link r_foot: geometry collision mesh filename=./meshes/r_foot_chull.obj; visual mesh filename=./meshes/r_foot.obj
